Commit message: basic_control: single-loop resolved-rate controller with layered src/
Restructure src/ into app/control/hardware/math layers. Replace the
reactive servo with a 100 Hz resolved-rate controller: Pinocchio
FK/Jacobian, damped least squares (Dls.h), velocity-to-position
integration commanded in POSITION mode, per-joint speed clipping from
Config.h, following-error guard, and FK arrival notice. Harden fault
handling (decoded faults, guarded restore, edge-triggered printing) and
add diagnose_faults tool, control-logic tests, and decision docs;
drop stale known-issues.md and CONTROLLER_CODE_MAP.md.

File: Christian_control/basic_control/config/GEN3_custom.urdf (robot description, URDF)
Before this commit: robot GEN3_URDF_V12, 10 links, 9 joints
Joints:
- joint Actuator1: limit effort=39 velocity=1.39 -> effort=39 velocity=1.3893
- joint Actuator2: limit lower=-2.41 upper=2.41 effort=39 velocity=1.39 -> lower=-2.41 upper=2.41 effort=39 velocity=1.3893
- joint Actuator3: limit effort=39 velocity=1.39 -> effort=39 velocity=1.3893
- joint Actuator4: limit lower=-2.66 upper=2.66 effort=39 velocity=1.39 -> lower=-2.66 upper=2.66 effort=39 velocity=1.3893
- joint Actuator5: limit effort=9 velocity=1.22 -> effort=9 velocity=1.2200
- joint Actuator6: limit lower=-2.23 upper=2.23 effort=9 velocity=1.22 -> lower=-2.23 upper=2.23 effort=9 velocity=1.2200
- joint Actuator7: limit effort=9 velocity=1.22 -> effort=9 velocity=1.2200
