Commit message: basic_control: land the rest of the in-progress refactor so HEAD builds
Completes the slice committed in 42579f58, which was an intermediate cut
that did not compile on its own. With these files HEAD builds standalone
and the full test suite passes from a clean checkout.

Contents, all pre-existing uncommitted working-tree work rather than part
of the no-motion/telemetry change:

  - Cyclic: command frame-id tracking (CyclicSession::last_command_frame_id),
    used by the format-5 log's command_frame_id column.
  - ServoingGuard: explicit Restore(std::ostream&) alongside the RAII
    retry, so a failed restore is visible rather than silent.
  - DualArmKinematics / Kinematics: mounted-model adapter updates; the
    right-base origin constant is now kRightBaseOriginControlM.
  - GEN3_dual_mounted.urdf: both chains realigned to Kinova's official
    ros_kortex v2.5.2 description. Joints 1/3/5/7 are continuous with no
    position range; 2/4/6 are revolute at +/-128.34 / 147.25 / 119.75 deg.
    Config.h kTrajectoryPosLimitDeg still reads 128.9 / 147.8 / 120.3 --
    the two agree on which joints are bounded and differ by ~0.55 deg,
    Config.h being the more permissive. Neither is this arm's CONFIGURED
    soft limit (README: j4 near -19.6 deg, j6 near +36 deg), which only
    the robot can confirm.
  - Controller/ReactiveLaw/ReactivePose/Target/TrajectoryFile, Connect:
    signature and header updates consistent with the above.
  - tests: replay_controller, test_playback, test_dual_arm_model,
    test_reactive_law, test_resolved_rate updated to the new signatures.
  - tools/query_limits.cpp removed (not referenced by any build target).
  - docs/: architecture, custom-urdf, reactive-pose-port,
    trajectory-playback, qdot-limit-raise, cartesian-velocity-controller.

Verified by materialising the staged index into a clean tree and building
it there: cmake --build -- 0 errors, ctest 7/7 passed.

CLAUDE.md is deliberately NOT included. Its working-tree edit deletes the
standing hardware-safety rules (the prohibition on running Kortex-linked
binaries without explicit authorization, and the presence/clear-workspace/
e-stop requirement), which is a policy change unrelated to making the
build work and should be committed on its own terms.

No hardware was connected; the arm was not moved.

File: Christian_control/basic_control/config/GEN3_dual_mounted.urdf (robot description, URDF)
Before this commit: robot GEN3_URDF_V12, 21 links, 20 joints
Links:
- link EndEffector_Link: mass None -> 0
- link leftEndEffector_Link: mass None -> 0
Joints:
- joint Actuator1: limit lower=-3.14 upper=3.14 effort=39 velocity=0.8727 -> effort=39 velocity=1.3963; type revolute -> continuous
- joint Actuator2: limit lower=-2.41 upper=2.41 effort=39 velocity=0.8727 -> lower=-2.24 upper=2.24 effort=39 velocity=1.3963
- joint Actuator3: limit lower=-3.14 upper=3.14 effort=39 velocity=0.8727 -> effort=39 velocity=1.3963; type revolute -> continuous
- joint Actuator4: limit lower=-2.66 upper=2.66 effort=39 velocity=0.8727 -> lower=-2.57 upper=2.57 effort=39 velocity=1.3963
- joint Actuator5: limit lower=-3.14 upper=3.14 effort=9 velocity=0.8727 -> effort=9 velocity=1.2218; type revolute -> continuous
- joint Actuator6: limit lower=-2.23 upper=2.23 effort=9 velocity=0.8727 -> lower=-2.09 upper=2.09 effort=9 velocity=1.2218
- joint Actuator7: limit lower=-3.14 upper=3.14 effort=9 velocity=0.8727 -> effort=9 velocity=1.2218; type revolute -> continuous
- joint leftActuator1: limit lower=-3.14 upper=3.14 effort=39 velocity=0.8727 -> effort=39 velocity=1.3963; type revolute -> continuous
- joint leftActuator2: limit lower=-2.41 upper=2.41 effort=39 velocity=0.8727 -> lower=-2.24 upper=2.24 effort=39 velocity=1.3963
- joint leftActuator3: limit lower=-3.14 upper=3.14 effort=39 velocity=0.8727 -> effort=39 velocity=1.3963; type revolute -> continuous
- joint leftActuator4: limit lower=-2.66 upper=2.66 effort=39 velocity=0.8727 -> lower=-2.57 upper=2.57 effort=39 velocity=1.3963
- joint leftActuator5: limit lower=-3.14 upper=3.14 effort=9 velocity=0.8727 -> effort=9 velocity=1.2218; type revolute -> continuous
- joint leftActuator6: limit lower=-2.23 upper=2.23 effort=9 velocity=0.8727 -> lower=-2.09 upper=2.09 effort=9 velocity=1.2218
- joint leftActuator7: limit lower=-3.14 upper=3.14 effort=9 velocity=0.8727 -> effort=9 velocity=1.2218; type revolute -> continuous

Commit message: controller: velocity-profiled targets, process-lock exclusivity, tool-frame FK fix
- Targets/Runner/Actuation: replace the fixed-target reach-sphere gate with
  a jerk-limited Cartesian trajectory profile from measured takeover pose to
  the compiled terminal target (TrajectoryProfile.h), so arrival no longer
  depends on a hardcoded distance bound.
- ProcessLock: exclusive filesystem-lock ownership of the controller
  resource, acquired before any hardware session is opened (Main.cpp).
- Kinematics: add AnalyticalKinematics, a closed-form Eigen-only FK chain
  independent of Pinocchio, cross-checked against Kinematics.cpp's URDF FK
  in test_analytical_kinematics (agree to <1e-9). Diff-verified this
  project's URDF against Kinova's official upstream GEN3-7DOF-VISION_ARM
  URDF_V12 and found the right-arm chain numerically identical.
- Fix a real FK/dashboard mismatch: the robot has a configured tool offset
  (ControlConfig::GetToolConfiguration, xyz 0 0 0.12 m) that no URDF can see.
  Added ConfiguredTool_Link to config/GEN3_dual_mounted.urdf and pointed
  config::kRightEndEffectorFrame at it, closing the gap between our FK and
  the Kinova dashboard's tool_pose from 0.12 m to 0.012 m.
- Hardware: expose Connect::control_config() (was already owned internally,
  only device_config() was exposed) so read-only tools can reach
  GetToolConfiguration without a duplicate client registration.
- New read-only diagnostic tools (no motion): print_joint_positions,
  print_end_effector_pose, print_tool_configuration,
  compare_end_effector_pose (firmware vs Pinocchio vs analytical FK, one
  shared feedback snapshot).
- docs/code-read and docs/decisions updated to match.

File: Christian_control/basic_control/config/GEN3_dual_mounted.urdf (robot description, URDF)
Before this commit: robot GEN3_URDF_V12, 21 links, 20 joints
Links:
- added link ConfiguredTool_Link, mass 0.831
Joints:
- added joint ConfiguredTool: type fixed, parent EndEffector_Link, child ConfiguredTool_Link, origin xyz=0 0 0.12 rpy=0 0 0, axis 0 0 0

Commit message: kinematics: world frame at the base midpoint, mounting geometry in YAML
The URDF already had a `world` root, but it sat 0.149614 m above the two
base_link origins: each arm was reached by rolling +-1.2085 rad and then
translating 0.16 m along the rolled y axis, through an intermediate
base_linktras / leftbase_linktras link. That put world equidistant from
both bases but not between them.

world now sits at the midpoint of the two base origins. Separation
(0.113415 m) and tilt (+-1.2085 rad) are unchanged - this is the same rig
re-expressed about a different origin. A URDF <origin> composes as
Trans(xyz) then Rot(rpy), verified empirically against Pinocchio rather
than assumed, so one fixed joint per arm now expresses each mount
directly. The intermediate links carried no geometry and are gone: frames
drop 44 -> 40, while nq=22 and nv=14 are untouched because every mounting
joint is fixed.

The numbers move into config/dual_arm_mounting.yaml, which is now their
declared source of truth. Nothing generates the URDF from it, so
test_dual_arm_mounting (ctest `dual_arm_mounting`) is the link between
them: it loads the URDF through the real Dynamics/DualArmKinematics path
and fails naming the number that disagrees. The values are INHERITED, not
measured - they arrived fully formed in af116a5c with no measurement note
and a round 0.16 m radius - and both the YAML and the decision record say
so, so a future survey has one place to change.

DualArmKinematics gains the world-frame layer this makes usable:
WorldFromBase, ToolPoseInWorld, FullConfiguration for both arms, and the
PointBaseToWorld / PointWorldToBase pair. These are ADDITIVE. `world` is
the URDF root, so Pinocchio's oMf placements already are world poses and
the base-frame methods are the ones doing extra work; ReactiveLaw, Safety
and the arrival monitors continue to reason in base_link axes, unchanged.

print_dual_arm_fk prints both arms in world and in their own base frames
for a chosen configuration. It links the URDF only, never Kortex, so it
cannot connect or command and is safe to run with the robot off. The two
tool frames are not the same point - ConfiguredTool_Link is right-arm
only - and every left figure is open-loop, both labelled as such.

Also flags createArmBasePoses (utils.cpp), which encodes a contradictory
mounting geometry (0.12058 m apart, rpy +-3pi/4) and is dead only because
its sole caller does not build.

File: Christian_control/basic_control/config/GEN3_dual_mounted.urdf (robot description, URDF)
Before this commit: robot GEN3_URDF_V12, 22 links, 21 joints
Links:
- removed link base_linktras
- removed link leftbase_linktras
Joints:
- removed joint left_base_rotation
- removed joint leftrot_linktras
- removed joint right_base_rotation
- removed joint rot_linktras
- added joint left_base_mount: type fixed, parent world, child leftbase_link, origin xyz=0 0.0567075 0 rpy=-1.2085 0 0
- added joint right_base_mount: type fixed, parent world, child base_link, origin xyz=0 -0.0567075 0 rpy=1.2085 0 0

Commit message: planner: Cartesian path tasks, deterministic IK, inter-arm clearance
Adds the ability to plan a traced Cartesian path (a circle) end to end, makes
planning reproducible, and adds inter-arm clearance checking. Point-to-point
behaviour is unchanged throughout (regression holds at 1.34181 mm).

Cartesian path planning
  A circle in goal.yaml is generated, seeded by continuation IK, optimised by
  GPMP2 with a per-waypoint pose prior, emitted, reconstructed with the
  CONTROLLER's own SampleJointTrajectory, densely validated, and released only
  if every modelled check passes. The approach phase is task-space
  unconstrained: the arm must reach the shape, but the route there was never
  part of the request.

  Validation runs on the reconstruction rather than the optimiser's output,
  because subsampling to the 1000-point wire cap and cubic-Hermite
  reconstruction both distort the plan AFTER optimisation finishes. Three
  errors are reported and one is gated: e_planner (desired vs GP-dense),
  e_command (desired vs 500 Hz reconstruction, GATED), and e_reconstruction
  (the transport loss between them), so a fidelity failure is attributable.

  Found doing this: GPMP2 interpolates with a constant support interval, so
  the two phases having different natural sample spacings emitted timestamps
  other than those requested. The validator then measured the approach as if
  it were the circle and reported 110 mm of error. Both phases now share one
  uniform grid, checked rather than assumed. 110 mm -> 2.4 mm.

Deterministic IK
  analytical_ik seeded from std::random_device, so identical requests planned
  differently: the traced circle was stable at 2.406-2.409 mm but closure
  drift swung 0.04-14 deg between runs. IKSeeding{seed, stream} replaces the
  function-local static generator (which advanced across calls, so even a
  fixed seed would have depended on call history). Streams keep exploration
  and determinism compatible: different restarts within a run, identical
  restarts across runs. Randomised mode remains for robustness testing but
  reports its drawn seed, so no run is unreproducible.

Inter-arm clearance
  InterArmDistanceChecker compares the two arms at CORRESPONDING TIMES over
  the start-skew window, not as a static swept volume: two arms passing
  through the same point ten seconds apart never meet, and activation is not
  atomic so identical local clocks cannot be assumed. Reports surface-to-
  surface clearance, both times, and the responsible sphere pair.

Also: pose-prior noise ordering is [rotation; translation] in one place,
pinned by a mutation-verified test; IK tolerance is a parameter of the request
rather than a property of the solver (its 20 mm early exit made path residuals
describe where the solver stopped, not where the arm can reach); planner.yaml
gains path_following and seeding sections under the existing strict loader.

Tests: planner_bridge 16/16, basic_control 11/11.

Not verified on hardware. modelled_collision_valid certifies against the arm
workspace plus an optional operator box only — no wearer, no torso, no second
arm — and every report says so.

File: Christian_control/basic_control/config/GEN3_dual_mounted.urdf (robot description, URDF)
Before this commit: robot GEN3_URDF_V12, 20 links, 19 joints
Links:
- removed link world
- added link mount
Joints:
- joint left_base_mount: parent world -> mount
- joint right_base_mount: parent world -> mount
