Commit message: chris

File: Christian_control/model/GEN3_dual_mounted.urdf (robot description, URDF)
Before this commit: robot GEN3_URDF_V12, 20 links, 19 joints
Links:
- removed link Bracelet_Link
- removed link ConfiguredTool_Link
- removed link EndEffector_Link
- removed link ForeArm_Link
- removed link HalfArm1_Link
- removed link HalfArm2_Link
- removed link Shoulder_Link
- removed link SphericalWrist1_Link
- removed link SphericalWrist2_Link
- removed link base_link
- removed link leftBracelet_Link
- removed link leftEndEffector_Link
- removed link leftForeArm_Link
- removed link leftHalfArm1_Link
- removed link leftHalfArm2_Link
- removed link leftShoulder_Link
- removed link leftSphericalWrist1_Link
- removed link leftSphericalWrist2_Link
- removed link leftbase_link
- added link left_base_link, mass 1.697; collision mesh filename=package://kortex_description/arms/gen3/7dof/meshes/base_lin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; visual mesh filename=package://kortex_description/arms/gen3/7dof/meshes/base_lin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
- added link left_bracelet_link, mass 0.5006; collision mesh filename=package://kortex_description/arms/gen3/7dof/meshes/bracelet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; visual mesh filename=package://kortex_description/arms/gen3/7dof/meshes/bracelet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
- added link left_end_effector_link, mass 0
- added link left_forearm_link, mass 0.9302; collision mesh filename=package://kortex_description/arms/gen3/7dof/meshes/forearm_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; visual mesh filename=package://kortex_description/arms/gen3/7dof/meshes/forearm_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
- added link left_half_arm_1_link, mass 1.1636; collision mesh filename=package://kortex_description/arms/gen3/7dof/meshes/half_arm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; visual mesh filename=package://kortex_description/arms/gen3/7dof/meshes/half_arm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
- added link left_half_arm_2_link, mass 1.1636; collision mesh filename=package://kortex_description/arms/gen3/7dof/meshes/half_arm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; visual mesh filename=package://kortex_description/arms/gen3/7dof/meshes/half_arm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
- added link left_shoulder_link, mass 1.3773; collision mesh filename=package://kortex_description/arms/gen3/7dof/meshes/shoulder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; visual mesh filename=package://kortex_description/arms/gen3/7dof/meshes/shoulder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
- added link left_spherical_wrist_1_link, mass 0.6781; collision mesh filename=package://kortex_description/arms/gen3/7dof/meshes/spherica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; visual mesh filename=package://kortex_description/arms/gen3/7dof/meshes/spherica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
- added link left_spherical_wrist_2_link, mass 0.6781; collision mesh filename=package://kortex_description/arms/gen3/7dof/meshes/spherica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; visual mesh filename=package://kortex_description/arms/gen3/7dof/meshes/spherica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
- added link left_tool_link, mass 0.831
- added link right_base_link, mass 1.697; collision mesh filename=package://kortex_description/arms/gen3/7dof/meshes/base_lin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; visual mesh filename=package://kortex_description/arms/gen3/7dof/meshes/base_lin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
- added link right_bracelet_link, mass 0.5006; collision mesh filename=package://kortex_description/arms/gen3/7dof/meshes/bracelet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; visual mesh filename=package://kortex_description/arms/gen3/7dof/meshes/bracelet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
- added link right_end_effector_link, mass 0
- added link right_forearm_link, mass 0.9302; collision mesh filename=package://kortex_description/arms/gen3/7dof/meshes/forearm_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; visual mesh filename=package://kortex_description/arms/gen3/7dof/meshes/forearm_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
- added link right_half_arm_1_link, mass 1.1636; collision mesh filename=package://kortex_description/arms/gen3/7dof/meshes/half_arm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; visual mesh filename=package://kortex_description/arms/gen3/7dof/meshes/half_arm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
- added link right_half_arm_2_link, mass 1.1636; collision mesh filename=package://kortex_description/arms/gen3/7dof/meshes/half_arm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; visual mesh filename=package://kortex_description/arms/gen3/7dof/meshes/half_arm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
- added link right_shoulder_link, mass 1.3773; collision mesh filename=package://kortex_description/arms/gen3/7dof/meshes/shoulder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; visual mesh filename=package://kortex_description/arms/gen3/7dof/meshes/shoulder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
- added link right_spherical_wrist_1_link, mass 0.6781; collision mesh filename=package://kortex_description/arms/gen3/7dof/meshes/spherica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; visual mesh filename=package://kortex_description/arms/gen3/7dof/meshes/spherica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
- added link right_spherical_wrist_2_link, mass 0.6781; collision mesh filename=package://kortex_description/arms/gen3/7dof/meshes/spherica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; visual mesh filename=package://kortex_description/arms/gen3/7dof/meshes/spherica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
- added link right_tool_link, mass 0.831
Joints:
- removed joint Actuator1
- removed joint Actuator2
- removed joint Actuator3
- removed joint Actuator4
- removed joint Actuator5
- removed joint Actuator6
- removed joint Actuator7
- removed joint ConfiguredTool
- removed joint EndEffector
- removed joint leftActuator1
- removed joint leftActuator2
- removed joint leftActuator3
- removed joint leftActuator4
- removed joint leftActuator5
- removed joint leftActuator6
- removed joint leftActuator7
- removed joint leftEndEffector
- removed joint left_base_mount
- removed joint right_base_mount
- added joint left_end_effector_fixed: type fixed, parent left_bracelet_link, child left_end_effector_link, origin xyz=0 0 -0.0615250000000001 rpy=3.14159265358979 1.09937075168372E-32 0, axis 0 0 0
- added joint left_joint_1: type continuous, parent left_base_link, child left_shoulder_link, origin xyz=0 0 0.15643 rpy=3.1416 2.7629E-18 -4.9305E-36, axis 0 0 1, limit effort=39 velocity=1.3963
- added joint left_joint_2: type revolute, parent left_shoulder_link, child left_half_arm_1_link, origin xyz=0 0.005375 -0.12838 rpy=1.5708 2.1343E-17 -1.1102E-16, axis 0 0 1, limit lower=-2.24 upper=2.24 effort=39 velocity=1.3963
- added joint left_joint_3: type continuous, parent left_half_arm_1_link, child left_half_arm_2_link, origin xyz=0 -0.21038 -0.006375 rpy=-1.5708 1.2326E-32 -2.9122E-16, axis 0 0 1, limit effort=39 velocity=1.3963
- added joint left_joint_4: type revolute, parent left_half_arm_2_link, child left_forearm_link, origin xyz=0 0.006375 -0.21038 rpy=1.5708 -6.6954E-17 -1.6653E-16, axis 0 0 1, limit lower=-2.57 upper=2.57 effort=39 velocity=1.3963
- added joint left_joint_5: type continuous, parent left_forearm_link, child left_spherical_wrist_1_link, origin xyz=0 -0.20843 -0.006375 rpy=-1.5708 2.2204E-16 -6.373E-17, axis 0 0 1, limit effort=9 velocity=1.2218
- added joint left_joint_6: type revolute, parent left_spherical_wrist_1_link, child left_spherical_wrist_2_link, origin xyz=0 0.00017505 -0.10593 rpy=1.5708 9.2076E-28 -8.2157E-15, axis 0 0 1, limit lower=-2.09 upper=2.09 effort=9 velocity=1.2218
- added joint left_joint_7: type continuous, parent left_spherical_wrist_2_link, child left_bracelet_link, origin xyz=0 -0.10593 -0.00017505 rpy=-1.5708 -5.5511E-17 9.6396E-17, axis 0 0 1, limit effort=9 velocity=1.2218
- added joint left_mount_to_base: type fixed, parent mount, child left_base_link, origin xyz=0 0.0375 0 rpy=-1.2085 0 0
- added joint left_tool_fixed: type fixed, parent left_end_effector_link, child left_tool_link, origin xyz=0 0 0.12 rpy=0 0 0, axis 0 0 0
- added joint right_end_effector_fixed: type fixed, parent right_bracelet_link, child right_end_effector_link, origin xyz=0 0 -0.0615250000000001 rpy=3.14159265358979 1.09937075168372E-32 0, axis 0 0 0
- added joint right_joint_1: type continuous, parent right_base_link, child right_shoulder_link, origin xyz=0 0 0.15643 rpy=3.1416 2.7629E-18 -4.9305E-36, axis 0 0 1, limit effort=39 velocity=1.3963
- added joint right_joint_2: type revolute, parent right_shoulder_link, child right_half_arm_1_link, origin xyz=0 0.005375 -0.12838 rpy=1.5708 2.1343E-17 -1.1102E-16, axis 0 0 1, limit lower=-2.24 upper=2.24 effort=39 velocity=1.3963
- added joint right_joint_3: type continuous, parent right_half_arm_1_link, child right_half_arm_2_link, origin xyz=0 -0.21038 -0.006375 rpy=-1.5708 1.2326E-32 -2.9122E-16, axis 0 0 1, limit effort=39 velocity=1.3963
- added joint right_joint_4: type revolute, parent right_half_arm_2_link, child right_forearm_link, origin xyz=0 0.006375 -0.21038 rpy=1.5708 -6.6954E-17 -1.6653E-16, axis 0 0 1, limit lower=-2.57 upper=2.57 effort=39 velocity=1.3963
- added joint right_joint_5: type continuous, parent right_forearm_link, child right_spherical_wrist_1_link, origin xyz=0 -0.20843 -0.006375 rpy=-1.5708 2.2204E-16 -6.373E-17, axis 0 0 1, limit effort=9 velocity=1.2218
- added joint right_joint_6: type revolute, parent right_spherical_wrist_1_link, child right_spherical_wrist_2_link, origin xyz=0 0.00017505 -0.10593 rpy=1.5708 9.2076E-28 -8.2157E-15, axis 0 0 1, limit lower=-2.09 upper=2.09 effort=9 velocity=1.2218
- added joint right_joint_7: type continuous, parent right_spherical_wrist_2_link, child right_bracelet_link, origin xyz=0 -0.10593 -0.00017505 rpy=-1.5708 -5.5511E-17 9.6396E-17, axis 0 0 1, limit effort=9 velocity=1.2218
- added joint right_mount_to_base: type fixed, parent mount, child right_base_link, origin xyz=0 -0.0375 0 rpy=1.2085 0 0
- added joint right_tool_fixed: type fixed, parent right_end_effector_link, child right_tool_link, origin xyz=0 0 0.12 rpy=0 0 0, axis 0 0 0
